File: tally/tally.kicad_pcb (KiCad board)
At the start: 2 copper layers, 71.8 x 30.5 mm, 11 parts, among them J1 Console, J2 Raspberry_Pi_2_3, U1 LP5009PWR

Commit message: forgotten update
Parts:
- R5: value 75 -> 160
Connections:
- J2 pad 11: (no net) -> Net-(J2-Pad11)
- J2 pad 12: (no net) -> Net-(J2-Pad12)
- J2 pad 13: (no net) -> Net-(J2-Pad13)
- J2 pad 15: (no net) -> Net-(J2-Pad15)
- J2 pad 16: (no net) -> Net-(J2-Pad16)
- J2 pad 18: (no net) -> Net-(J2-Pad18)
- J2 pad 19: (no net) -> Net-(J2-Pad19)
- J2 pad 21: (no net) -> Net-(J2-Pad21)
- J2 pad 22: (no net) -> Net-(J2-Pad22)
- J2 pad 23: (no net) -> Net-(J2-Pad23)
- J2 pad 24: (no net) -> Net-(J2-Pad24)
- J2 pad 26: (no net) -> Net-(J2-Pad26)
- J2 pad 27: (no net) -> Net-(J2-Pad27)
- J2 pad 28: (no net) -> Net-(J2-Pad28)
- J2 pad 29: (no net) -> Net-(J2-Pad29)
- J2 pad 31: (no net) -> Net-(J2-Pad31)
- J2 pad 32: (no net) -> Net-(J2-Pad32)
- J2 pad 33: (no net) -> Net-(J2-Pad33)
- J2 pad 35: (no net) -> Net-(J2-Pad35)
- J2 pad 36: (no net) -> Net-(J2-Pad36)
- J2 pad 37: (no net) -> Net-(J2-Pad37)
- J2 pad 38: (no net) -> Net-(J2-Pad38)
- J2 pad 40: (no net) -> Net-(J2-Pad40)
- J2 pad 7: (no net) -> Net-(J2-Pad7)
