File: tally/tally.sch (KiCad schematic (older format))
At the start: 11 parts, among them J1 Console, J2 Raspberry_Pi_2_3, U1 LP5009PWR

Commit message: forgotten update
Parts:
- R5: value 75 -> 160
Changed lines of the file:
@@
 P 6200 3500
 F 0 "R5" H 6259 3546 50  0000 L CNN
-F 1 "75" H 6259 3455 50  0000 L CNN
+F 1 "160" H 6259 3455 50  0000 L CNN
 F 2 "Resistor_SMD:R_1206_3216Metric_Pad1.30x1.75mm_HandSolder" H 6200 3500 50  0001 C CNN
 F 3 "~" H 6200 3500 50  0001 C CNN
